File: hardware/SYNTH_01.kicad_pcb (KiCad board)
At the start: 2 copper layers, 112.7 x 150 mm, 100 parts, among them J2 Conn_01x04_Pin, SW1 SW_Push_45deg, SW10 SW_Push_45deg, SW11 SW_Push_45deg, SW12 SW_Push_45deg, SW13 SW_Push_45deg, SW14 SW_Push_45deg, SW15 SW_Push_45deg, SW16 SW_Push_45deg, SW17 SW_Push_45deg, SW18 SW_Push_45deg, SW19 SW_Push_45deg, SW2 SW_Push_45deg, SW20 SW_Push_45deg, SW21 SW_Push_45deg, SW3 SW_Push_45deg, SW4 SW_Push_45deg, SW5 SW_Push_45deg, SW6 SW_Push_45deg, SW7 SW_Push_45deg, SW8 SW_Push_45deg, SW9 SW_Push_45deg, U1 MCP23017-E/SP, U2 74AHCT1G125

Commit message: PCB REFACTOR : need to finish connecting isolated GND areas
Routing:
- net /SYNTH_01/COL2: track 0.00 -> 383.9 mm, vias 0 -> 1
- net /SYNTH_01/COL1: track 0.00 -> 316.1 mm, vias 0 -> 2
- net /SYNTH_01/ROW4: track 0.00 -> 274.2 mm
- net /SYNTH_01/COL3: track 0.00 -> 253.9 mm, vias 0 -> 9
- net /SYNTH_01/COL_SHIFT: track 0.00 -> 235.7 mm, vias 0 -> 1
- net /SYNTH_01/COL0: track 0.00 -> 211.4 mm, vias 0 -> 1
- net /SYNTH_01/ROW3: track 0.00 -> 195.9 mm, vias 0 -> 1
- net /SYNTH_01/ROW2: track 0.00 -> 177.7 mm
- net GND: track 206.8 -> 383.4 mm, vias 21 -> 24
- net /SYNTH_01/ROW1: track 0.00 -> 123.0 mm, vias 0 -> 1
- net /SYNTH_01/ROW0: track 0.00 -> 104.5 mm, vias 0 -> 3
- net Net-(D21-A): track 0.00 -> 16.3 mm
- net Net-(D1-A): track 0.00 -> 14.6 mm
- net Net-(D3-A): track 0.00 -> 14.6 mm
- net Net-(D2-A): track 0.00 -> 14.6 mm
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Other:
- board text added: "AKOR_01 [PCB] Arthur Kowskii Croquebois August 2026"

Commit message: PCB REFACTOR: finish corrected LED routing
Parts:
- D22, D23, D24, D25, D26, D27, D28, D29, D30, D31, D32, D33, D34, D35, D36, D37, D38, D39, D40, D41: moved to B.Cu
- turned D22 to 180 degrees
- turned D23 to 180 degrees
- turned D24 to 180 degrees
- turned D25 to 180 degrees
- turned D26 to 0 degrees
- turned D27 to 0 degrees
- turned D28 to 0 degrees
- turned D29 to 0 degrees
- turned D30 to 180 degrees
- turned D31 to 180 degrees
- turned D32 to 180 degrees
- turned D33 to 180 degrees
- turned D34 to 0 degrees
- turned D35 to 0 degrees
- turned D36 to 0 degrees
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Routing:
- net LED_5V: track 928.7 -> 415.5 mm, vias 0 -> 20
- net /SYNTH_01/E2_SW: track 0.00 -> 346.1 mm, vias 0 -> 1
- net /SYNTH_01/E1_SW: track 0.00 -> 323.9 mm, vias 0 -> 1
- net /SYNTH_01/E4_SW: track 0.00 -> 150.2 mm, vias 0 -> 3
- net /SYNTH_01/E3_SW: track 0.00 -> 146.2 mm, vias 0 -> 1
- net +3V3: track 0.00 -> 141.1 mm
- net /SYNTH_01/E7_SW: track 0.00 -> 131.2 mm
- net /SYNTH_01/SDA: track 0.00 -> 121.7 mm
- net /SYNTH_01/SCL: track 0.00 -> 109.5 mm
- net /SYNTH_01/E1_B: track 0.00 -> 105.1 mm
- net /SYNTH_01/E1_A: track 0.00 -> 103.7 mm
- net /SYNTH_01/E5_SW: track 0.00 -> 100.7 mm, vias 0 -> 5
- net Net-(U1-~{RESET}): track 0.00 -> 99.8 mm
- net /SYNTH_01/E3_A: track 0.00 -> 90.4 mm, vias 0 -> 1
- net /SYNTH_01/E2_B: track 0.00 -> 87.8 mm
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- added copper zone on In1.Cu, net GND
- added copper zone on In2.Cu, net GND
- added copper zone on F.Cu, net LED_5V
- removed copper zone on B.Cu, net GND
Other:
- copper layers 2 -> 4
