File: hardware/AKOR_01.kicad_pcb (KiCad board)
At the start: 4 copper layers, 112.7 x 150 mm, 100 parts, among them J2 Conn_01x04_Pin, SW1 SW_Push_45deg, SW10 SW_Push_45deg, SW11 SW_Push_45deg, SW12 SW_Push_45deg, SW13 SW_Push_45deg, SW14 SW_Push_45deg, SW15 SW_Push_45deg, SW16 SW_Push_45deg, SW17 SW_Push_45deg, SW18 SW_Push_45deg, SW19 SW_Push_45deg, SW2 SW_Push_45deg, SW20 SW_Push_45deg, SW21 SW_Push_45deg, SW3 SW_Push_45deg, SW4 SW_Push_45deg, SW5 SW_Push_45deg, SW6 SW_Push_45deg, SW7 SW_Push_45deg, SW8 SW_Push_45deg, SW9 SW_Push_45deg, U1 MCP23017-E/SP, U2 74AHCT1G125

Commit message: Rename project to AKOR_01
Connections:
- net /SYNTH_01/COL0 renamed /AKOR_01/COL0
- net /SYNTH_01/COL1 renamed /AKOR_01/COL1
- net /SYNTH_01/COL2 renamed /AKOR_01/COL2
- net /SYNTH_01/COL3 renamed /AKOR_01/COL3
- net /SYNTH_01/COL_SHIFT renamed /AKOR_01/COL_SHIFT
- net /SYNTH_01/E1_A renamed /AKOR_01/E1_A
- net /SYNTH_01/E1_B renamed /AKOR_01/E1_B
- net /SYNTH_01/E1_SW renamed /AKOR_01/E1_SW
- net /SYNTH_01/E2_A renamed /AKOR_01/E2_A
- net /SYNTH_01/E2_B renamed /AKOR_01/E2_B
- net /SYNTH_01/E2_SW renamed /AKOR_01/E2_SW
- net /SYNTH_01/E3_A renamed /AKOR_01/E3_A
- net /SYNTH_01/E3_B renamed /AKOR_01/E3_B
- net /SYNTH_01/E3_SW renamed /AKOR_01/E3_SW
- net /SYNTH_01/E4_A renamed /AKOR_01/E4_A
- net /SYNTH_01/E4_B renamed /AKOR_01/E4_B
- net /SYNTH_01/E4_SW renamed /AKOR_01/E4_SW
- net /SYNTH_01/E5_A renamed /AKOR_01/E5_A
- net /SYNTH_01/E5_B renamed /AKOR_01/E5_B
- net /SYNTH_01/E5_SW renamed /AKOR_01/E5_SW
- net /SYNTH_01/E6_A renamed /AKOR_01/E6_A
- net /SYNTH_01/E6_B renamed /AKOR_01/E6_B
- net /SYNTH_01/E6_SW renamed /AKOR_01/E6_SW
- net /SYNTH_01/E7_A renamed /AKOR_01/E7_A
- net /SYNTH_01/E7_B renamed /AKOR_01/E7_B
- net /SYNTH_01/E7_SW renamed /AKOR_01/E7_SW
- net /SYNTH_01/ROW0 renamed /AKOR_01/ROW0
- net /SYNTH_01/ROW1 renamed /AKOR_01/ROW1
- net /SYNTH_01/ROW2 renamed /AKOR_01/ROW2
- net /SYNTH_01/ROW3 renamed /AKOR_01/ROW3
- net /SYNTH_01/ROW4 renamed /AKOR_01/ROW4
- net /SYNTH_01/SCL renamed /AKOR_01/SCL
- net /SYNTH_01/SDA renamed /AKOR_01/SDA
